Commit message: path planning in physical robot and control in sim

File: src/panda_test/urdf/panda_arm_encoderless_vs.xacro (robot description, xacro)
@@ -16,18 +16,18 @@
     <link name="world"/>
         <!-- Red Circle Definition -->
-    <link name="red_obstacle">
+    <!-- <link name="red_obstacle">
         <visual>
             <geometry>
-                <cylinder length="0.01" radius="0.1"/> <!-- Adjust size as needed -->
+                <cylinder length="0.01" radius="0.1"/>
             </geometry>
             <material name="red"/>
         </visual>
-    </link>
-    <joint name="red_circle_joint" type="fixed">
-        <origin xyz="0.5 0 0.5" rpy="1.57 0 0"/> <!-- Adjust position relative to the world or robot -->
-        <parent link="${arm_id}_link0"/> <!-- or another reference link, e.g., a link of the robot -->
+    </link> -->
+    <!-- <joint name="red_circle_joint" type="fixed">
+        <origin xyz="0.25 0 0.9" rpy="1.57 0 0"/>
+        <parent link="${arm_id}_link0"/>
         <child link="red_obstacle"/>
         <axis xyz="0 0 0"/>
-    </joint>
+    </joint>    -->
     <joint name="fixed" type="fixed">
       <origin rpy="0 0 0" xyz="0.00 0.00 0.00"/>

Commit message: added franka_control and dual learning rate

File: src/panda_test/urdf/panda_arm_encoderless_vs.xacro (robot description, xacro)
@@ -47,7 +47,12 @@
       </collision>
       <inertial>
-        <mass value="0.1" />
-        <inertia ixx="0.03" iyy="0.03" izz="0.03" ixy="0.0" ixz="0.0" iyz="0.0" />
-      </inertial>
+        <!-- <mass value="0.1" /> -->
+        <mass value="0.629769273993887"/>
+        <inertia ixx="0.3" iyy="0.3" izz="0.3" ixy="0.0" ixz="0.0" iyz="0.0" />
+      </inertial>
+      <!-- <inertial>
+        <mass value="0.629769273993887"/>
+        <inertia ixx="0.0031531502307724" ixy="8.29043977620386E-07" ixz="0.000153878135879635" iyy="0.00388160500528917" iyz="8.22996985150111E-06" izz="0.00428506837339653"/>
+      </inertial> -->
     </link>
     <link name="${arm_id}_link1">
@@ -63,6 +68,8 @@
       </collision>
       <inertial>
-        <mass value="0.1" />
-        <inertia ixx="0.03" iyy="0.03" izz="0.03" ixy="0.0" ixz="0.0" iyz="0.0" />
+        <!-- <mass value="0.1" /> -->
+        <inertia ixx="0.3" iyy="0.3" izz="0.3" ixy="0.0" ixz="0.0" iyz="0.0" />
+        <mass value="4.970684"/>
+        <!-- <inertia ixx="0.70337" ixy="-0.00013900" ixz="0.0067720" iyy="0.70661" iyz="0.019169" izz="0.0091170"/> -->
       </inertial>
     </link>
@@ -87,6 +94,8 @@
       </collision>
       <inertial>
-        <mass value="0.1" />
-        <inertia ixx="0.03" iyy="0.03" izz="0.03" ixy="0.0" ixz="0.0" iyz="0.0" />
+        <!-- <mass value="0.1" /> -->
+        <inertia ixx="0.3" iyy="0.3" izz="0.3" ixy="0.0" ixz="0.0" iyz="0.0" />
+        <mass value="0.646926"/>
+        <!-- <inertia ixx="0.0079620" ixy="-3.9250e-3" ixz="1.0254e-02" iyy="2.8110e-02" iyz="7.0400e-04" izz="2.5995e-02"/> -->
       </inertial>
     </link>
@@ -111,6 +120,8 @@
       </collision>
       <inertial>
-        <mass value="0.1" />
-        <inertia ixx="0.03" iyy="0.03" izz="0.03" ixy="0.0" ixz="0.0" iyz="0.0" />
+        <!-- <mass value="0.1" /> -->
+        <inertia ixx="0.3" iyy="0.3" izz="0.3" ixy="0.0" ixz="0.0" iyz="0.0" />
+        <mass value="3.228604"/>
+        <!-- <inertia ixx="3.7242e-02" ixy="-4.7610e-03" ixz="-1.1396e-02" iyy="3.6155e-02" iyz="-1.2805e-02" izz="1.0830e-02"/> -->
       </inertial>
     </link>
@@ -135,6 +146,8 @@
       </collision>
       <inertial>
-        <mass value="0.1" />
-        <inertia ixx="0.03" iyy="0.03" izz="0.03" ixy="0.0" ixz="0.0" iyz="0.0" />
+        <!-- <mass value="0.1" /> -->
+        <inertia ixx="0.3" iyy="0.3" izz="0.3" ixy="0.0" ixz="0.0" iyz="0.0" />
+        <mass value="3.587895"/>
+        <!-- <inertia ixx="2.5853e-02" ixy="7.7960e-03" ixz="-1.3320e-03" iyy="1.9552e-02" iyz="8.6410e-03" izz="2.8323e-02"/> -->
       </inertial>
     </link>
@@ -159,6 +172,8 @@
       </collision>
       <inertial>
-        <mass value="0.1" />
-        <inertia ixx="0.03" iyy="0.03" izz="0.03" ixy="0.0" ixz="0.0" iyz="0.0" />
+        <!-- <mass value="0.1" /> -->
+        <inertia ixx="0.3" iyy="0.3" izz="0.3" ixy="0.0" ixz="0.0" iyz="0.0" />
+        <mass value="1.225946"/>
+        <!-- <inertia ixx="3.5549e-02" ixy="-2.1170e-03" ixz="-4.0370e-03" iyy="2.9474e-02" iyz="2.2900e-04" izz="8.6270e-03"/> -->
       </inertial>
     </link>
@@ -183,6 +198,8 @@
       </collision>
       <inertial>
-        <mass value="0.1" />
-        <inertia ixx="0.03" iyy="0.03" izz="0.03" ixy="0.0" ixz="0.0" iyz="0.0" />
+        <!-- <mass value="0.1" /> -->
+        <inertia ixx="0.3" iyy="0.3" izz="0.3" ixy="0.0" ixz="0.0" iyz="0.0" />
+        <mass value="1.666555"/>
+        <!-- <inertia ixx="1.9640e-03" ixy="1.0900e-04" ixz="-1.1580e-03" iyy="4.3540e-03" iyz="3.4100e-04" izz="5.4330e-03"/> -->
       </inertial>
     </link>
@@ -207,6 +224,8 @@
       </collision>
       <inertial>
-        <mass value="0.1" />
-        <inertia ixx="0.03" iyy="0.03" izz="0.03" ixy="0.0" ixz="0.0" iyz="0.0" />
+        <!-- <mass value="0.1" /> -->
+        <inertia ixx="0.3" iyy="0.3" izz="0.3" ixy="0.0" ixz="0.0" iyz="0.0" />
+        <mass value="7.35522e-01"/>
+        <!-- <inertia ixx="1.2516e-02" ixy="-4.2800e-04" ixz="-1.1960e-03" iyy="1.0027e-02" iyz="-7.4100e-04" izz="4.8150e-03"/> -->
       </inertial>
     </link>
